Commit message: add inertia in gp7

File: src/description/motoman_gp7/motoman_gp7_support/urdf/gp7_macro.xacro (robot description, xacro)
@@ -3,4 +3,5 @@
 <xacro:macro name="motoman_gp7" params="prefix">
     <xacro:include filename="$(find motoman_resources)/urdf/common_materials.xacro"/>
+    <xacro:include filename="$(find xacro_inertia)/urdf/inertia_table.xacro"/>
     <!-- link list -->
     <link name="${prefix}base_link">
@@ -16,4 +17,7 @@
             </geometry>
         </collision>
+        <inertial>
+            <xacro:cylinder_inertia m="8" r="0.095" h="0.15"/>
+        </inertial>
     </link>
     <link name="${prefix}link_1_s">
@@ -29,4 +33,7 @@
             </geometry>
         </collision>
+        <inertial>
+            <xacro:cylinder_inertia m="5" r="0.095" h="0.18"/>
+        </inertial>
     </link>
     <link name="${prefix}link_2_l">
@@ -42,4 +49,7 @@
             </geometry>
         </collision>
+        <inertial>
+            <xacro:cylinder_inertia m="10" r="0.095" h="0.26"/>
+        </inertial>
     </link>
     <link name="${prefix}link_3_u">
@@ -55,4 +65,7 @@
             </geometry>
         </collision>
+        <inertial>
+            <xacro:cylinder_inertia m="4" r="0.095" h="0.1"/>
+        </inertial>
     </link>
     <link name="${prefix}link_4_r">
@@ -68,4 +81,7 @@
             </geometry>
         </collision>
+        <inertial>
+            <xacro:cylinder_inertia m="6" r="0.095" h="0.19"/>
+        </inertial>
     </link>
     <link name="${prefix}link_5_b">
@@ -81,4 +97,7 @@
             </geometry>
         </collision>
+        <inertial>
+            <xacro:cylinder_inertia m="3" r="0.095" h="0.1"/>
+        </inertial>
     </link>
     <link name="${prefix}link_6_t">
@@ -94,4 +113,7 @@
             </geometry>
         </collision>
+        <inertial>
+            <xacro:cylinder_inertia m="2" r="0.095" h="0.072"/>
+        </inertial>
     </link>
     <link name="${prefix}tool0"/>
