Commit message: gp7 from git

File: src/description/cogniman_scene_description/urdf/robot.urdf (robot description, URDF)
Before this commit: robot cogniman_robot, 12 links, 11 joints
Links:
- added link base
- link base_link: mass 0.008 -> None; geometry collision mesh filename=package://motoman_gp7_support/meshes/collision/gp7_base_lin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; visual mesh filename=package://motoman_gp7_support/meshes/visual/gp7_base_link.s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
- link link_1_s: mass 0.005 -> None; geometry collision mesh filename=package://motoman_gp7_support/meshes/collision/gp7_link_1_s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; visual mesh filename=package://motoman_gp7_support/meshes/visual/gp7_link_1_s.stl
- link link_2_l: mass 0.01 -> None; geometry collision mesh filename=package://motoman_gp7_support/meshes/collision/gp7_link_2_l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; visual mesh filename=package://motoman_gp7_support/meshes/visual/gp7_link_2_l.stl
- link link_3_u: mass 0.004 -> None; geometry collision mesh filename=package://motoman_gp7_support/meshes/collision/gp7_link_3_u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; visual mesh filename=package://motoman_gp7_support/meshes/visual/gp7_link_3_u.stl
- link link_4_r: mass 0.006 -> None; geometry collision mesh filename=package://motoman_gp7_support/meshes/collision/gp7_link_4_r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; visual mesh filename=package://motoman_gp7_support/meshes/visual/gp7_link_4_r.stl
- link link_5_b: mass 0.003 -> None; geometry collision mesh filename=package://motoman_gp7_support/meshes/collision/gp7_link_5_b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; visual mesh filename=package://motoman_gp7_support/meshes/visual/gp7_link_5_b.stl
- link link_6_t: mass 0.002 -> None; geometry collision mesh filename=package://motoman_gp7_support/meshes/collision/gp7_link_6_t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; visual mesh filename=package://motoman_gp7_support/meshes/visual/gp7_link_6_t.stl
Joints:
- added joint base_link-base: type fixed, parent base_link, child base, origin xyz=0 0 0.330 rpy=0 0 0
- joint joint_1_s: limit lower=-1.9 upper=1.9 effort=212.66 velocity=6.5448 -> lower=-2.9670 upper=2.9670 effort=212.66 velocity=6.5448
- joint joint_2_l: limit lower=-1.1 upper=1.47 effort=205.80 velocity=5.4977 -> lower=-1.1344 upper=2.5307 effort=205.80 velocity=5.4977
- joint joint_3_u: limit lower=-1.2 upper=3.2 effort=106.82 velocity=7.1558 -> lower=-1.2217 upper=3.3161 effort=106.82 velocity=7.1558
- joint joint_4_r: limit lower=-3.0 upper=3.0 effort=55.86 velocity=9.5993 -> lower=-3.3161 upper=3.3161 effort=55.86 velocity=9.5993
- joint joint_5_b: limit lower=-2.34 upper=2.34 effort=32.68 velocity=9.5993 -> lower=-2.3561 upper=2.3561 effort=32.68 velocity=9.5993
- joint joint_6_t: limit lower=-6.2 upper=6.2 effort=22.54 velocity=17.4845 -> lower=-6.2944 upper=6.2944 effort=22.54 velocity=17.4845

File: src/description/motoman_gp7/motoman_gp7_support/urdf/gp7_macro.xacro (robot description, xacro)
@@ -3,10 +3,9 @@
 <xacro:macro name="motoman_gp7" params="prefix">
     <xacro:include filename="$(find motoman_resources)/urdf/common_materials.xacro"/>
-    <xacro:include filename="$(find motoman_gp7_support)/urdf/inertia_description/inertia_table.xacro"/>
     <!-- link list -->
     <link name="${prefix}base_link">
         <visual>
             <geometry>
-                <mesh filename="file:///$(find motoman_gp7_support)/meshes/visual/gp7_base_link.stl"/>
+                <mesh filename="package://motoman_gp7_support/meshes/visual/gp7_base_link.stl"/>
             </geometry>
             <xacro:material_yaskawa_blue/>
@@ -14,18 +13,12 @@
         <collision>
             <geometry>
-                <mesh filename="file:///$(find motoman_gp7_support)/meshes/collision/gp7_base_link.stl"/>
+                <mesh filename="package://motoman_gp7_support/meshes/collision/gp7_base_link.stl"/>
             </geometry>
         </collision>
-        <inertial>
-            <xacro:cylinder_inertia m="8" r="0.095" h="0.15"/>
-        </inertial>
     </link>
-    <gazebo reference="${prefix}base_link">
-        <material>Gazebo/Blue</material>
-    </gazebo>
     <link name="${prefix}link_1_s">
         <visual>
             <geometry>
-                <mesh filename="file:///$(find motoman_gp7_support)/meshes/visual/gp7_link_1_s.stl"/>
+                <mesh filename="package://motoman_gp7_support/meshes/visual/gp7_link_1_s.stl"/>
             </geometry>
             <xacro:material_yaskawa_blue/>
@@ -33,38 +26,12 @@
         <collision>
             <geometry>
-                <mesh filename="file:///$(find motoman_gp7_support)/meshes/collision/gp7_link_1_s.stl"/>
+                <mesh filename="package://motoman_gp7_support/meshes/collision/gp7_link_1_s.stl"/>
             </geometry>
         </collision>
-        <inertial>
-            <xacro:cylinder_inertia m="5" r="0.095" h="0.18"/>
-        </inertial>
     </link>
-    <gazebo reference="${prefix}link_1_s">
-        <material>Gazebo/Blue</material>
-    </gazebo>
     <link name="${prefix}link_2_l">
         <visual>
             <geometry>
-                <mesh filename="file:///$(find motoman_gp7_support)/meshes/visual/gp7_link_2_l.stl"/>
-            </geometry>
-            <xacro:material_yaskawa_blue/>
-        </visual>
-        <collision>
-            <origin xyz="-0.03 -0.0 -0.33" rpy="${pi/2} 0.0 ${-pi/2}" />
-            <geometry>
-                <mesh filename="file:///$(find motoman_gp7_support)/meshes/collision/gp7_link_2_l.stl" scale = "0.001 0.001 0.001"/>
-            </geometry>
-        </collision>
-        <inertial>
-            <xacro:cylinder_inertia m="10" r="0.095" h="0.26"/>
-        </inertial>
-    </link>
-    <gazebo reference="${prefix}link_2_l">
-        <material>Gazebo/Blue</material>
-    </gazebo>
-    <link name="${prefix}link_3_u">
-        <visual>
-            <geometry>
-                <mesh filename="file:///$(find motoman_gp7_support)/meshes/visual/gp7_link_3_u.stl"/>
+                <mesh filename="package://motoman_gp7_support/meshes/visual/gp7_link_2_l.stl"/>
             </geometry>
             <xacro:material_yaskawa_blue/>
@@ -72,18 +39,12 @@
         <collision>
             <geometry>
-                <mesh filename="file:///$(find motoman_gp7_support)/meshes/collision/gp7_link_3_u.stl"/>
+                <mesh filename="package://motoman_gp7_support/meshes/collision/gp7_link_2_l.stl"/>
             </geometry>
         </collision>
-        <inertial>
-            <xacro:cylinder_inertia m="4" r="0.095" h="0.1"/>
-        </inertial>
     </link>
-    <gazebo reference="${prefix}link_3_u">
-        <material>Gazebo/Blue</material>
-    </gazebo>
-    <link name="${prefix}link_4_r">
+    <link name="${prefix}link_3_u">
         <visual>
             <geometry>
-                <mesh filename="file:///$(find motoman_gp7_support)/meshes/visual/gp7_link_4_r.stl"/>
+                <mesh filename="package://motoman_gp7_support/meshes/visual/gp7_link_3_u.stl"/>
             </geometry>
             <xacro:material_yaskawa_blue/>
@@ -91,18 +52,12 @@
         <collision>
             <geometry>
-                <mesh filename="file:///$(find motoman_gp7_support)/meshes/collision/gp7_link_4_r.stl"/>
+                <mesh filename="package://motoman_gp7_support/meshes/collision/gp7_link_3_u.stl"/>
             </geometry>
         </collision>
-        <inertial>
-            <xacro:cylinder_inertia m="6" r="0.095" h="0.19"/>
-        </inertial>
     </link>
-    <gazebo reference="${prefix}link_4_r">
-        <material>Gazebo/Blue</material>
-    </gazebo>
-    <link name="${prefix}link_5_b">
+    <link name="${prefix}link_4_r">
         <visual>
             <geometry>
-                <mesh filename="file:///$(find motoman_gp7_support)/meshes/visual/gp7_link_5_b.stl"/>
+                <mesh filename="package://motoman_gp7_support/meshes/visual/gp7_link_4_r.stl"/>
             </geometry>
             <xacro:material_yaskawa_blue/>
@@ -110,18 +65,12 @@
         <collision>
             <geometry>
-                <mesh filename="file:///$(find motoman_gp7_support)/meshes/collision/gp7_link_5_b.stl"/>
+                <mesh filename="package://motoman_gp7_support/meshes/collision/gp7_link_4_r.stl"/>
             </geometry>
         </collision>
-        <inertial>
-            <xacro:cylinder_inertia m="3" r="0.095" h="0.1"/>
-        </inertial>
     </link>
-    <gazebo reference="${prefix}link_5_b">
-        <material>Gazebo/Blue</material>
-    </gazebo>
-    <link name="${prefix}link_6_t">
+    <link name="${prefix}link_5_b">
         <visual>
             <geometry>
-                <mesh filename="file:///$(find motoman_gp7_support)/meshes/visual/gp7_link_6_t.stl"/>
+                <mesh filename="package://motoman_gp7_support/meshes/visual/gp7_link_5_b.stl"/>
             </geometry>
             <xacro:material_yaskawa_blue/>
@@ -129,14 +78,21 @@
         <collision>
             <geometry>
-                <mesh filename="file:///$(find motoman_gp7_support)/meshes/collision/gp7_link_6_t.stl"/>
+                <mesh filename="package://motoman_gp7_support/meshes/collision/gp7_link_5_b.stl"/>
             </geometry>
         </collision>
-        <inertial>
-            <xacro:cylinder_inertia m="2" r="0.095" h="0.072"/>
-        </inertial>
     </link>
-    <gazebo reference="${prefix}link_6_t">
-        <material>Gazebo/Blue</material>
-    </gazebo>
+    <link name="${prefix}link_6_t">
+        <visual>
+            <geometry>
+                <mesh filename="package://motoman_gp7_support/meshes/visual/gp7_link_6_t.stl"/>
+            </geometry>
+            <xacro:material_yaskawa_blue/>
+        </visual>
+        <collision>
+            <geometry>
+                <mesh filename="package://motoman_gp7_support/meshes/collision/gp7_link_6_t.stl"/>
+            </geometry>
+        </collision>
+    </link>
     <link name="${prefix}tool0"/>
     <!-- end of link list -->
@@ -147,5 +103,5 @@
         <origin xyz="0 0 0.330" rpy="0 0 0" />
         <axis xyz="0 0 1" />
-        <limit lower="-1.9" upper="1.9" effort="212.66" velocity="6.5448"/>
+        <limit lower="-2.9670" upper="2.9670" effort="212.66" velocity="6.5448"/>
     </joint>
     <joint name="${prefix}joint_2_l" type="revolute">
@@ -154,5 +110,5 @@
         <origin xyz="0.040 0 0" rpy="0 0 0" />
         <axis xyz="0 1 0" />
-        <limit lower="-1.1" upper="1.47" effort="205.80" velocity="5.4977"/>
+        <limit lower="-1.1344" upper="2.5307" effort="205.80" velocity="5.4977"/>
     </joint>
     <joint name="${prefix}joint_3_u" type="revolute">
@@ -161,5 +117,5 @@
         <origin xyz="0 0 0.445" rpy="0 0 0" />
         <axis xyz="0 -1 0" />
-        <limit lower="-1.2" upper="3.2" effort="106.82" velocity="7.1558"/>
+        <limit lower="-1.2217" upper="3.3161" effort="106.82" velocity="7.1558"/>
     </joint>
     <joint name="${prefix}joint_4_r" type="revolute">
@@ -168,5 +124,5 @@
         <origin xyz="0.440 0 0.040" rpy="0 0 0" />
         <axis xyz="-1 0 0" />
-        <limit lower="-3.0" upper="3.0" effort="55.86" velocity="9.5993"/>
+        <limit lower="-3.3161" upper="3.3161" effort="55.86" velocity="9.5993"/>
     </joint>
     <joint name="${prefix}joint_5_b" type="revolute">
@@ -175,5 +131,5 @@
         <origin xyz="0 0 0" rpy="0 0 0" />
         <axis xyz="0 -1 0" />
-        <limit lower="-2.34" upper="2.34" effort="32.68" velocity="9.5993"/>
+        <limit lower="-2.3561" upper="2.3561" effort="32.68" velocity="9.5993"/>
     </joint>
     <joint name="${prefix}joint_6_t" type="revolute">
@@ -182,5 +138,5 @@
         <origin xyz="0 0 0" rpy="0 0 0" />
         <axis xyz="-1 0 0" />
-        <limit lower="-6.2" upper="6.2" effort="22.54" velocity="17.4845"/>
+        <limit lower="-6.2944" upper="6.2944" effort="22.54" velocity="17.4845"/>
     </joint>
     <joint name="${prefix}joint_6_t-tool0" type="fixed">
@@ -191,10 +147,10 @@
     <!-- end of joint list -->
     <!-- ROS base_link to Robot Manufacturer World Coordinates transform -->
-    <!-- <link name="${prefix}base" />
+    <link name="${prefix}base" />
     <joint name="${prefix}base_link-base" type="fixed">
         <origin xyz="0 0 0.330" rpy="0 0 0"/>
         <parent link="${prefix}base_link"/>
         <child link="${prefix}base"/>
-    </joint> -->
+    </joint>
     </xacro:macro>
 </robot>

Commit message: add joint state from gazebo (plugin and bridge)

File: src/description/cogniman_scene_description/urdf/robot.urdf (robot description, URDF)
Before this commit: robot cogniman_robot, 19 links, 18 joints
Joints:
- joint robot_to_profilo: origin xyz=0 0 0 rpy=0 0 0 -> xyz=0.3 1 0 rpy=0 0 0
