Commit message: added gripper clamp ad positionning in urdf

File: src/description/cogniman_scene_description/urdf/cogniman_description.xacro (robot description, xacro)
@@ -1,3 +1,8 @@
 <robot xmlns:xacro="http://ros.org/wiki/xacro" name="cogniman_robot">
+    <xacro:include filename="$(find screw_gripper_description)/urdf/screw_gripper.xacro"/>
+    <xacro:include filename="$(find positionning_tool)/urdf/positionning_tool.xacro"/>
+    <xacro:equerre prefix="1"/>
+    <xacro:equerre prefix="2"/>
+    <xacro:equerre prefix="3"/>
     <xacro:include filename="$(find toggle_clamp)/urdf/toggle_clamp.xacro"/>
     <xacro:clamp prefix="1"/>
@@ -7,23 +12,46 @@
 	<xacro:motoman_gp7 prefix=""/>
     <link name="world"/>
-    <joint name="world_to_plateforme" type="fixed">
-        <origin xyz="1 0 0" rpy="0 0 0"/>
+    <joint name="world_to_robot" type="fixed">
+        <origin xyz="0 0 0.24" rpy="0 0 0"/>
         <parent link="world"/>
+        <child link="base_link"/>
+    </joint>
+    <joint name="robot_to_plateforme" type="fixed">
+        <origin xyz="0 0 0" rpy="0 0 3.14"/>
+        <parent link="base_link"/>
         <child link="plateforme"/>
     </joint>
-    <joint name="plateforme_to_robot" type="fixed">
-        <origin xyz="1 0 0" rpy="0 0 0"/>
-        <parent link="plateforme"/>
-        <child link="base_link"/>
+    <!-- ======  TOOL ====== -->
+    <joint name="tool0_to_screw_gripper" type="fixed">
+        <origin xyz="0 0 0" rpy="0 0 0"/>
+        <parent link="tool0"/>
+        <child link="screw_gripper"/>
     </joint>
+    <!-- ======  CLAMP ====== -->
     <joint name="robot_to_clamp1" type="fixed">
-        <origin xyz="0 0 0" rpy="0 0 0"/>
+        <origin xyz="0.5 0.5 0" rpy="0 0 0"/>
         <parent link="base_link"/>
         <child link="clamp_1"/>
     </joint>
-       <joint name="robot_to_clamp2" type="fixed">
-        <origin xyz="0 0 0" rpy="0 0 0"/>
+    <joint name="robot_to_clamp2" type="fixed">
+        <origin xyz="0.2 0.2 0" rpy="0 0 0"/>
         <parent link="base_link"/>
         <child link="clamp_2"/>
     </joint>
+    <!-- ======  EQUERRE ====== -->
+    <joint name="robot_to_equerre1" type="fixed">
+        <origin xyz="1 1 0" rpy="0 0 0"/>
+        <parent link="base_link"/>
+        <child link="equerre_1"/>
+    </joint>
+        <joint name="robot_to_equerre2" type="fixed">
+        <origin xyz="1 1.2 0" rpy="0 0 0"/>
+        <parent link="base_link"/>
+        <child link="equerre_2"/>
+    </joint>
+        <joint name="robot_to_equerre3" type="fixed">
+        <origin xyz="1 1.5 0" rpy="0 0 0"/>
+        <parent link="base_link"/>
+        <child link="equerre_3"/>
+    </joint>
 </robot>

File: src/description/cogniman_scene_description/urdf/robot.urdf (robot description, URDF)
Before this commit: robot cogniman_robot, 13 links, 12 joints
Links:
- added link equerre_1; collision mesh filename=package://positionning_tool/mesh/collision/equerre_collisio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; visual mesh filename=package://positionning_tool/mesh/visual/equerre.stl
- added link equerre_2; collision mesh filename=package://positionning_tool/mesh/collision/equerre_collisio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; visual mesh filename=package://positionning_tool/mesh/visual/equerre.stl
- added link equerre_3; collision mesh filename=package://positionning_tool/mesh/collision/equerre_collisio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; visual mesh filename=package://positionning_tool/mesh/visual/equerre.stl
- added link screw_gripper; collision mesh filename=package://screw_gripper_description/mesh/collision/screw_gr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; visual mesh filename=package://screw_gripper_description/mesh/visual/screw_gripp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
- added link tcp_screw_gripper
Joints:
- removed joint plateforme_to_robot
- removed joint world_to_plateforme
- added joint robot_to_equerre1: type fixed, parent base_link, child equerre_1, origin xyz=1 1 0 rpy=0 0 0
- added joint robot_to_equerre2: type fixed, parent base_link, child equerre_2, origin xyz=1 1.2 0 rpy=0 0 0
- added joint robot_to_equerre3: type fixed, parent base_link, child equerre_3, origin xyz=1 1.5 0 rpy=0 0 0
- added joint robot_to_plateforme: type fixed, parent base_link, child plateforme, origin xyz=0 0 0 rpy=0 0 3.14
- added joint screw_gripper_to_tcp: type fixed, parent screw_gripper, child tcp_screw_gripper, origin xyz=0 0 0.2 rpy=0 0 0
- added joint tool0_to_screw_gripper: type fixed, parent tool0, child screw_gripper, origin xyz=0 0 0 rpy=0 0 0
- added joint world_to_robot: type fixed, parent world, child base_link, origin xyz=0 0 0.24 rpy=0 0 0
- joint robot_to_clamp1: origin xyz=0 0 0 rpy=0 0 0 -> xyz=0.5 0.5 0 rpy=0 0 0
- joint robot_to_clamp2: origin xyz=0 0 0 rpy=0 0 0 -> xyz=0.2 0.2 0 rpy=0 0 0

Commit message: added inertia to mototman (wrong value)

File: src/description/cogniman_scene_description/urdf/cogniman_description.xacro (robot description, xacro)
@@ -9,6 +9,6 @@
     <xacro:clamp prefix="2"/>
     <xacro:include filename="$(find plateforme_description)/urdf/plateforme.xacro"/>
-    <xacro:include filename="$(find motoman_gp7_support)/urdf/gp7_macro.xacro" />
-	<xacro:motoman_gp7 prefix=""/>
+    <xacro:include filename="$(find motoman_gp7_with_inertia)/urdf/gp7_with_inertia.xacro" />
+	<xacro:motoman_gp7_with_inertia prefix=""/>
     <link name="world"/>
     <joint name="world_to_robot" type="fixed">

File: src/description/cogniman_scene_description/urdf/robot.urdf (robot description, URDF)
Before this commit: robot cogniman_robot, 18 links, 17 joints
Links:
- link base_link: mass None -> 8; geometry 
- link link_1_s: mass None -> 5; geometry 
- link link_2_l: mass None -> 8; geometry 
- link link_3_u: mass None -> 4; geometry 
- link link_4_r: mass None -> 0.3; geometry 
- link link_5_b: mass None -> 2; geometry 
- link link_6_t: mass None -> 1; geometry 
- link tool0: mass None -> 1

Commit message: added profilo

File: src/description/cogniman_scene_description/urdf/cogniman_description.xacro (robot description, xacro)
@@ -1,2 +1,3 @@
+<?xml version="1.0" ?>
 <robot xmlns:xacro="http://ros.org/wiki/xacro" name="cogniman_robot">
     <xacro:include filename="$(find screw_gripper_description)/urdf/screw_gripper.xacro"/>
@@ -8,4 +9,5 @@
     <xacro:clamp prefix="1"/>
     <xacro:clamp prefix="2"/>
+    <xacro:include filename="$(find profilo_description)/urdf/profilo_with_support.xacro"/>
     <xacro:include filename="$(find plateforme_description)/urdf/plateforme.xacro"/>
     <xacro:include filename="$(find motoman_gp7_support)/urdf/gp7_macro.xacro" />
@@ -14,4 +16,5 @@
     <!-- <xacro:motoman_gp7_with_inertia prefix=""/> -->
     <link name="world"/>
+    <!-- ======  ROBOT ====== -->
     <joint name="world_to_robot" type="fixed">
         <origin xyz="0 0 0.24" rpy="0 0 0"/>
@@ -19,8 +22,15 @@
         <child link="base_link"/>
     </joint>
+    <!-- ======  PLATEFORME ====== -->
     <joint name="robot_to_plateforme" type="fixed">
         <origin xyz="0 0 0" rpy="0 0 3.14"/>
         <parent link="base_link"/>
         <child link="plateforme"/>
+    </joint>
+    <!-- ======  PROFILO ====== -->
+    <joint name="robot_to_profilo" type="fixed">
+        <origin xyz="0 0 0" rpy="0 0 0"/>
+        <parent link="base_link"/>
+        <child link="profilo"/>
     </joint>
     <!-- ======  TOOL ====== -->

File: src/description/cogniman_scene_description/urdf/robot.urdf (robot description, URDF)
Before this commit: robot cogniman_robot, 18 links, 17 joints
Links:
- added link profilo; collision mesh filename=package://profilo_description/mesh/collision/profilo_with_s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; visual mesh filename=package://profilo_description/mesh/visual/profilo_with_supp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
- link base_link: geometry collision mesh filename=package://motoman_gp7_support/meshes/collision/gp7_base_lin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; visual mesh filename=package://motoman_gp7_support/meshes/visual/gp7_base_link.s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
- link link_1_s: geometry collision mesh filename=package://motoman_gp7_support/meshes/collision/gp7_link_1_s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; visual mesh filename=package://motoman_gp7_support/meshes/visual/gp7_link_1_s.stl
- link link_2_l: mass 8 -> 10; geometry collision mesh filename=package://motoman_gp7_support/meshes/collision/gp7_link_2_l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; visual mesh filename=package://motoman_gp7_support/meshes/visual/gp7_link_2_l.stl
- link link_3_u: geometry collision mesh filename=package://motoman_gp7_support/meshes/collision/gp7_link_3_u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; visual mesh filename=package://motoman_gp7_support/meshes/visual/gp7_link_3_u.stl
- link link_4_r: mass 0.3 -> 6; geometry collision mesh filename=package://motoman_gp7_support/meshes/collision/gp7_link_4_r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; visual mesh filename=package://motoman_gp7_support/meshes/visual/gp7_link_4_r.stl
- link link_5_b: mass 2 -> 3; geometry collision mesh filename=package://motoman_gp7_support/meshes/collision/gp7_link_5_b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; visual mesh filename=package://motoman_gp7_support/meshes/visual/gp7_link_5_b.stl
- link link_6_t: mass 1 -> 2; geometry collision mesh filename=package://motoman_gp7_support/meshes/collision/gp7_link_6_t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; visual mesh filename=package://motoman_gp7_support/meshes/visual/gp7_link_6_t.stl
- link tool0: mass 1 -> None
Joints:
- added joint robot_to_profilo: type fixed, parent base_link, child profilo, origin xyz=0 0 0 rpy=0 0 0

Commit message: change profilo position

File: src/description/cogniman_scene_description/urdf/cogniman_description.xacro (robot description, xacro)
@@ -1,4 +1,5 @@
 <?xml version="1.0" ?>
 <robot xmlns:xacro="http://ros.org/wiki/xacro" name="cogniman_robot">
+    <xacro:include filename="$(find cogniman_scene_description)/urdf/cogniman_gazebo.xacro"/>
     <xacro:include filename="$(find screw_gripper_description)/urdf/screw_gripper.xacro"/>
     <xacro:include filename="$(find positionning_tool)/urdf/positionning_tool.xacro"/>
@@ -30,5 +31,5 @@
     <!-- ======  PROFILO ====== -->
     <joint name="robot_to_profilo" type="fixed">
-        <origin xyz="0 0 0" rpy="0 0 0"/>
+        <origin xyz="0.3 1 0" rpy="0 0 0"/>
         <parent link="base_link"/>
         <child link="profilo"/>

Commit message: .

File: src/description/cogniman_scene_description/urdf/cogniman_description.xacro (robot description, xacro)
@@ -10,5 +10,5 @@
     </plugin>
     </gazebo>
-    <!-- <xacro:include filename="$(find cogniman_scene_description)/urdf/cogniman_gazebo.xacro"/> -->
+    <xacro:include filename="$(find cogniman_scene_description)/urdf/cogniman_gazebo.xacro"/>
     <xacro:include filename="$(find screw_gripper_description)/urdf/screw_gripper.xacro"/>
     <xacro:include filename="$(find positionning_tool)/urdf/positionning_tool.xacro"/>

File: src/description/cogniman_scene_description/urdf/cogniman_gazebo.xacro (robot description, xacro)
@@ -1,17 +1,15 @@
 <?xml version="1.0" ?>
 <robot xmlns:xacro="http://ros.org/wiki/xacro" name="cogniman_gazebo">
-    <gazebo>
-        <physics name="10ms" type="ode">
-            <max_step_size>0.01</max_step_size>
-            <real_time_factor>1.0</real_time_factor>
-        </physics>
-        <plugin
-            filename="gz-sim-physics-system"
-            name="gz::sim::systems::Physics">
-        </plugin>
-        <plugin filename="libgazebo_ros_control.so" name="gazebo_ros_control">
-            <robotNamespace>/</robotNamespace>
-            <robotParam>/robot_description</robotParam>
-        </plugin>
-    </gazebo>
+ <gazebo reference="joint_6_t-tool0">
+    <sensor name="force_torque_sensor" type="force_torque">
+      <always_on>true</always_on>
+      <update_rate>50</update_rate>
+      <visualize>true</visualize>
+      <topic>tool0/force_torque</topic>
+      <force_torque>
+        <frame>sensor</frame>
+        <measure_direction>parent_to_child</measure_direction>
+      </force_torque>
+    </sensor>
+  </gazebo>
 </robot>

File: src/description/cogniman_scene_description/urdf/robot.urdf (robot description, URDF)
Before this commit: robot cogniman_robot, 19 links, 18 joints
Links:
- link clamp_1: mass None -> 0.6
- link clamp_2: mass None -> 0.6
- link equerre_1: mass None -> 0.5
- link equerre_2: mass None -> 0.5
- link equerre_3: mass None -> 0.5
- link plateforme: mass None -> 200
- link profilo: mass None -> 4
- link screw_gripper: mass None -> 0.5

Commit message: add tcp in urdf

File: src/description/cogniman_scene_description/urdf/cogniman_description.xacro (robot description, xacro)
@@ -26,4 +26,11 @@
     <!-- <xacro:motoman_gp7_with_inertia prefix=""/> -->
     <link name="world"/>
+    <link name="tcp"/>
+    <!-- ======  TCP ====== -->
+    <joint name="tool0_to_tcp" type="fixed">
+        <origin xyz="0 0 0" rpy="0 0 0"/>
+        <parent link="tool0"/>
+        <child link="tcp"/>
+    </joint>
     <!-- ======  ROBOT ====== -->
     <joint name="world_to_robot" type="fixed">
