Commit message: add inertia

File: src/description/plateforme_description/urdf/plateforme.xacro (robot description, xacro)
@@ -1,4 +1,6 @@
+<?xml version="1.0" ?>
 <robot xmlns:xacro="http://ros.org/wiki/xacro">
     <xacro:include filename="$(find xacro_materials)/urdf/materials.xacro"/>
+    <xacro:include filename="$(find xacro_inertia)/urdf/inertia_table.xacro"/>
     <link name="plateforme">
         <visual>
@@ -13,4 +15,7 @@
             </geometry>
         </collision>
+        <inertial>
+          <xacro:box_inertia m="200" x="2" y="1" z="0.25"/>
+        </inertial>
     </link>
 </robot>

File: src/description/positionning_tool/urdf/positionning_tool.xacro (robot description, xacro)
@@ -1,4 +1,6 @@
+<?xml version="1.0" ?>
 <robot xmlns:xacro="http://ros.org/wiki/xacro">
     <xacro:macro name="equerre" params="prefix">
+    <xacro:include filename="$(find xacro_inertia)/urdf/inertia_table.xacro"/>
     <xacro:include filename="$(find xacro_materials)/urdf/materials.xacro"/>
     <link name="equerre_${prefix}">
@@ -14,4 +16,7 @@
             </geometry>
         </collision>
+        <inertial>
+          <xacro:box_inertia m="0.5" x="0.05" y="0.05" z="0.05"/>
+        </inertial>
     </link>
     </xacro:macro>

File: src/description/profilo_description/urdf/profilo_with_support.xacro (robot description, xacro)
@@ -2,4 +2,5 @@
 <robot xmlns:xacro="http://ros.org/wiki/xacro">
     <!-- <xacro:macro name="profilo_with_support" params="prefix"> -->
+    <xacro:include filename="$(find xacro_inertia)/urdf/inertia_table.xacro"/>
     <xacro:include filename="$(find xacro_materials)/urdf/materials.xacro"/>
     <link name="profilo">
@@ -15,4 +16,7 @@
             </geometry>
         </collision>
+        <inertial>
+          <xacro:box_inertia m="4" x="0.05" y="0.05" z="0.05"/>
+        </inertial>
     </link>
     <!-- </xacro:macro> -->

File: src/description/screw_gripper_description/urdf/screw_gripper.xacro (robot description, xacro)
@@ -1,4 +1,6 @@
+<?xml version="1.0" ?>
 <robot xmlns:xacro="http://ros.org/wiki/xacro">
     <xacro:include filename="$(find xacro_materials)/urdf/materials.xacro"/>
+    <xacro:include filename="$(find xacro_inertia)/urdf/inertia_table.xacro"/>
     <link name="screw_gripper">
         <visual>
@@ -13,4 +15,7 @@
             </geometry>
         </collision>
+        <inertial>
+          <xacro:box_inertia m="0.5" x="0.05" y="0.15" z="0.05"/>
+        </inertial>
     </link>
     <link name="tcp_screw_gripper"/>

File: src/description/toggle_clamp/urdf/toggle_clamp.xacro (robot description, xacro)
@@ -1,5 +1,7 @@
+<?xml version="1.0" ?>
 <robot xmlns:xacro="http://ros.org/wiki/xacro">
     <xacro:macro name="clamp" params="prefix">
     <xacro:include filename="$(find xacro_materials)/urdf/materials.xacro"/>
+    <xacro:include filename="$(find xacro_inertia)/urdf/inertia_table.xacro"/>
     <link name="clamp_${prefix}">
         <visual>
@@ -14,4 +16,7 @@
             </geometry>
         </collision>
+        <inertial>
+          <xacro:box_inertia m="0.6" x="0.05" y="0.15" z="0.05"/>
+        </inertial>
     </link>
     </xacro:macro>
